File: BSPD/BSPD-revamp/BPSD-2025/BPSD-2025.kicad_sch (KiCad schematic)
At the start: 33 parts, among them J1 Conn(BSE_1), J2 Conn(BSE_2), J5 Conn(12V), J6 Conn(Hall Effect), U104 R-78E5.0-0.5, U2 LM339, U3 74AUC2G32, U4 74AUC2G08, U5 LM339

Commit message: BSPD Stuff
Parts:
- added C10: 100uF, symbol Device:C
- added Q1: PMOS, symbol Simulation_SPICE:PMOS
- added R1, R14, R15, R16, R17, R5: 100k, symbol Device:R_US
- added R11, R12, R13: 100k, Resistor_SMD:R_0603_1608Metric, symbol Device:R_US
- added R18: 2.2k, Resistor_SMD:R_0603_1608Metric, symbol Device:R_US
- added R19, R4: 10k, symbol Device:R_US
- added R2: 41, symbol Device:R_US
- added R20: 1k, Resistor_SMD:R_0603_1608Metric, symbol Device:R_US
- added R3: 1k, symbol Device:R_US
- added U1, U6, U9: LM339, symbol Comparator:LM339
- added U10: 74AUC2G32, symbol 74xGxx:74AUC2G32
- added U11: 74AUC2G08, symbol 74xGxx:74AUC2G08
- added U12: 74AHC1G32, symbol 74xGxx:74AHC1G32
- added unit 1 of U5
- added U7: 74AHC1G08, symbol 74xGxx:74AHC1G08
- added U8: 74AHC1G00, symbol 74xGxx:74AHC1G00
- C4: value 0.1uF -> 100uF
Connections:
- net +12V: now also Q1.1 (D)
- net +5V: now also R11.1, R12.1, R13.1, R15.2, R17.2, R4.1, R5.2, U12.5 (VCC), U7.5 (VCC), U8.5 (VCC)
- net BSE_1: now also R14.1, U5.5 (+), U9.11 (+)
- net BSE_2: now also R16.1, U6.5 (+), U9.9 (+)
- net BSPD_OUT: now also Q1.3 (S), R19.1
- net GND: now also C10.2, R1.2, R14.2, R16.2, R19.2, R2.2, R3.2, U12.3 (GND), U7.3 (GND), U8.3 (GND)
- net THRESH_ACCUM: now also U9.4 (-)
- net THRESH_BSE: now also U9.10 (-), U9.8 (-)
- net ACCUM_V renamed ACCUM_CURRENT
- net ACCUM_CURRENT: now also R1.1, R2.1, U1.5 (+), U9.5 (+); no longer C4.1
- new net: C4.1, R18.2, U12.2
- new net: R11.2, U11.1, U9.2
- new net: R12.2, U10.5, U9.13
- new net: R15.1, U5.2, U7.1
- new net: R17.1, U6.2, U7.2
- new net: U7.4, U8.2
- new net: R5.1, U1.2, U8.1
- new net: R20.1, U8.4
- new net: C10.1, R20.2, U12.1
- new net: R13.2, U10.6, U9.14
- new net: R18.1, U11.7
- new net: U10.3, U11.2
- new net 0.455V: R3.1, R4.2, U1.4 (-), U5.4 (-), U6.4 (-)
Other:
- note added: "τ = 0.22s"
- moved on the sheet: C3, C7, C8, C9, R10, R6, R7, R8, R9, TP4, TP5, TP6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
