File: BreathOf_fresh_Air/BreathOf_fresh_Air.kicad_sch (KiCad schematic)
At the start: 8 parts, among them J1 436500225, J2 436500428, U1 LM7805MPX/NOPB, U2 ALDP105W

Commit message: finished schematic and layout
Parts:
- removed C1, C2: C, symbol Device:C
- removed D1: 1N4001, Diode_THT:D_DO-41_SOD81_P10.16mm_Horizontal, symbol Diode:1N4001
- removed J1: 436500225, CONN_SD-43650-009_02_MOL, symbol 43650-0225:436500225
- removed R1: R_US, symbol Device:R_US
- added C1: CGA2B3X7R1E224K050BB, CAP_1005_TDK, symbol CGA2B3X7R1E224K050BB:CGA2B3X7R1E224K050BB
- added C2: CL21B224KAFNNNE, CAP_CL21_SAM, symbol CL21B224KAFNNNE:CL21B224KAFNNNE
- added CR1: 1N4148WX-TP, CR_SOD323_MCC, symbol 1N4148WX-TP:1N4148WX-TP
- added J3: 436500227, CONN_SD-43650-010_02_MOL, symbol 436500227:436500227
- added R1: CRCW040210K0FKED, RES_CRCW_0402, symbol CRCW040210K0FKED:CRCW040210K0FKED
Connections:
- net +12V: now also J2.4, C2.1; no longer J2.1
- net +5V: now also U2.1, C1.2, CR1.2, R1.2; no longer U2.4
- net FAN_ENABLE: now also J2.2, U2.4, CR1.1; no longer J2.3, U2.1
- net FAN_GND: now also J3.1
- net FAN_PWM: now also J2.3, J3.2, R1.1; no longer J2.4
- net GND: now also J2.1, C1.1, C2.2; no longer J2.2
