File: Fault Latch/Fault Latch 2.kicad_sch (KiCad schematic)
At the start: 113 parts, among them J1 1053141312, J3 1053131202, J4 1053131202, J5 1053131202, K3 Fujitsu_FTR-LYCA005x, K5 Fujitsu_FTR-LYCA005x, K6 Fujitsu_FTR-LYCA005x, Q101 Q_NPN_BEC, Q102 Q_NPN_BEC, Q103 Q_NPN_BEC, Q104 Q_NPN_BEC, Q105 Q_NMOS_GSD, Q106 Q_NMOS_GSD, Q110 Q_NPN_BEC, Q111 Q_NPN_BEC, Q112 Q_NMOS_GSD, Q113 Q_NMOS_GSD, Q114 Q_NMOS_GSD, Q115 Q_NMOS_GSD, Q117 Q_NMOS_GSD, Q118 Q_NMOS_GSD, Q119 Q_NMOS_GSD, Q120 Q_NMOS_GSD, Q121 Q_NMOS_GSD, Q122 Q_NMOS_GSD, Q123 Q_NMOS_GSD, Q124 Q_NMOS_GSD, Q125 Q_NMOS_GSD, SW101 SW_Omron_B3FS, SW102 SW_Omron_B3FS, SW103 SW_Omron_B3FS, U1 74LS279, U104 74AHC1G00, U109 74AHC1G00, U112 74AHC1G00, U117 74AHC1G00, U118 LM555xM, U2 LM1117DT-5.0, U7 SN74AHC1G08DBVR, U8 SN74AHC1G08DBVR

Commit message: Almost finished Fault Latch Layout Spring Semester V2.0
Parts:
- removed C102, C119, C120: 100n, Capacitor_SMD:C_0603_1608Metric_Pad1.08x0.95mm_HandSolder, symbol Device:C
- removed C110: 0.1u, Capacitor_SMD:C_0402_1005Metric, symbol Device:C
- removed J5: 1053131202, Connector_Molex:Molex_Nano-Fit_105313-xx02_1x02_P2.50mm_Horizontal, symbol molex.2-pin:1053131202
- removed K3, K5, K6: Fujitsu_FTR-LYCA005x, Relay_THT:Relay_SPDT_Fujitsu_FTR-LYCA005x_FormC_Vertical, symbol Relay:Fujitsu_FTR-LYCA005x
- removed Q119, Q121, Q122, Q123, Q124, Q125: Q_NMOS_GSD, Package_TO_SOT_SMD:SOT-23, symbol Transistor_FET:Q_NMOS_GSD
- removed R106, R107, R109, R116, R126, R134: 1k, Resistor_SMD:R_0805_2012Metric_Pad1.20x1.40mm_HandSolder, symbol Device:R_US
- removed R138, R139, R140: 10k, Resistor_SMD:R_0805_2012Metric_Pad1.20x1.40mm_HandSolder, symbol Device:R_US
- removed U104, U109, U112, U117: 74AHC1G00, Package_TO_SOT_SMD:SOT-23-5, symbol 74xGxx:74AHC1G00
- removed U3: ~, Package_TO_SOT_SMD:SOT-223, symbol New_Library:BTS4141NHUMA1_
- added C1: 100n, Capacitor_SMD:C_0603_1608Metric_Pad1.08x0.95mm_HandSolder, symbol Device:C
- added K1, K2, K3: Relay_SPDT_Omron_G2RL-1, Relay_THT:Relay_SPDT_Omron_G2RL-1, symbol Relay:G2RL-1
- added R1, R6, R7: 1k, Resistor_SMD:R_0805_2012Metric_Pad1.20x1.40mm_HandSolder, symbol Device:R_US
- added R2, R5, R8: 10k, Resistor_SMD:R_0805_2012Metric_Pad1.20x1.40mm_HandSolder, symbol Device:R_US
- added U2, U4, U5: SFH617A-1, Package_DIP:DIP-4_W7.62mm, symbol Isolator:SFH617A-1
- added U6: 74HCT00, symbol 74xx:74HCT00
- H101, H102, H103, H104: footprint MountingHole:MountingHole_3.2mm_M3 -> MountingHole:MountingHole_4.3mm_M4
- U1: footprint Package_SO:SOIC-16_3.9x9.9mm_P1.27mm -> Package_DIP:DIP-16_W7.62mm
Connections:
- net +12V: now also D104.1 (K), D108.1 (K), D110.1 (K), K1.A1, K2.A1, K3.A1, R7.1, U2.1, U4.1
- net +5V: now also C1.1, R1.1, R6.1, U5.4, U6.14 (VCC); no longer D104.1 (K), D108.1 (K), D110.1 (K)
- net BMS_SR: now also U6.13
- net BSPD_HV: now also R5.1, U4.2
- net GND: now also C1.2, R2.2, R5.2, R8.2, U2.3, U4.3, U6.7 (GND)
- net IMD_HV: now also R2.1, U2.2
- net IMD_SR: now also U6.12
- net NBMS_HV: now also U5.2
- net NBMS_LV: now also R8.1, U5.3, U6.1
- net NBPSD_LV: now also R6.2, U4.4, U6.9
- net NRESET_BMS: now also U6.2
- net NRESET_BSPD: now also U6.10
- net NRESET_IMD: now also U6.5
- net Shutdown Circuit In: now also K1.14
- net Shutdown Circuit Out: now also K3.11
- net at TP4.1: now also K1.11, K2.14
- net at D104.2 (A), Q117.3 (D): now also K1.A2
- net at D108.2 (A), Q118.3 (D): now also K2.A2
- net at U7.1: now also U6.11
- net at U1.6 (~{S}): now also U6.6
- net at TP11.1: now also K2.11, K3.14
- net at U1.11 (~{S}), U1.12 (~{S}): now also U6.8
- net at D110.2 (A), Q120.3 (D): now also K3.A2
- net at U1.2 (~{S}), U1.3 (~{S}): now also U6.3
- new net: R7.2, U5.1
- new net: R1.2, U2.4, U6.4
- no-connect marks 6 -> 7
Other:
- note added: "BMS Floating when faulted"
- moved on the sheet: C107, C108, C109, C111, C112, C113, C114, C115, C116, C118, D102, D104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

Commit message: Bom + Schematic Redone V3.2
Parts:
- removed C113: 47u, Capacitor_SMD:CP_Elec_6.3x5.4, symbol Device:C
- removed C114: 1u, Capacitor_SMD:C_0805_2012Metric_Pad1.18x1.45mm_HandSolder, symbol Device:C
- removed C115: 0.33u, Capacitor_SMD:C_0603_1608Metric_Pad1.08x0.95mm_HandSolder, symbol Device:C
- removed C116: 100n, Capacitor_SMD:C_0603_1608Metric_Pad1.08x0.95mm_HandSolder, symbol Device:C
- removed U2: LM1117DT-5.0, Package_TO_SOT_SMD:TO-252-3_TabPin2, symbol Regulator_Linear:LM1117DT-5.0
- added PS1: SCWN06A-05, SCWN06A05, symbol 1.Custom:SCWN06A-05
- J1: footprint footprints:CONN_SD-105314-100_12_MOL -> Connector_Molex:Molex_Nano-Fit_105314-xx12_2x06_P2.50mm_Horizontal
- R1, R6, R7: footprint Resistor_SMD:R_0805_2012Metric_Pad1.20x1.40mm_HandSolder -> Resistor_SMD:R_1210_3225Metric; JLC# C2889437 -> C230096; MOUSER (none) -> AC1210FR-071KL
- R101, R110, R113, R119, R122, R127: footprint Resistor_SMD:R_0805_2012Metric_Pad1.20x1.40mm_HandSolder -> Resistor_SMD:R_1210_3225Metric; JLC# C149504 -> C230004; MOUSER (none) -> AC1210FR-07100KL
- R105, R114, R121, R123, R136, R2, R5, R8: footprint Resistor_SMD:R_0805_2012Metric_Pad1.20x1.40mm_HandSolder -> Resistor_SMD:R_1210_3225Metric; MOUSER ESR10EZPD1002 -> 603-RC1210JR-0710KL
- R108, R111, R115, R120, R124, R129: footprint Resistor_SMD:R_0805_2012Metric_Pad1.20x1.40mm_HandSolder -> Resistor_SMD:R_1210_3225Metric; JLC# C17513 -> C230096; MOUSER (none) -> AC1210FR-071KL
- R112, R135: footprint Resistor_SMD:R_0603_1608Metric -> Resistor_SMD:R_1210_3225Metric; JLC# KTR03EZPF5100 -> C230277; MOUSER KTR03EZPF5100 -> AC1210FR-07510RL
- R117, R128, R137: footprint Resistor_SMD:R_0805_2012Metric_Pad1.20x1.40mm_HandSolder -> Resistor_SMD:R_1210_3225Metric; JLC# C1359 -> C137097; MOUSER (none) -> RC1210FR-072KL
- R130: footprint Resistor_SMD:R_0603_1608Metric -> Resistor_SMD:R_1210_3225Metric; JLC# C4151887 -> C230144; MOUSER ESR03EZPF2700 -> AC1210FR-07270RL
- R131: footprint Resistor_SMD:R_0603_1608Metric -> Resistor_SMD:R_1210_3225Metric; JLC# C22809 -> C230040; MOUSER (none) -> AC1210FR-0715KL
- R132: footprint Resistor_SMD:R_0603_1608Metric -> Resistor_SMD:R_1210_3225Metric; JLC# C60491 -> C230004; MOUSER (none) -> AC1210FR-07100KL
- R133: footprint Resistor_SMD:R_0805_2012Metric -> Resistor_SMD:R_1210_3225Metric; JLC# C1359 -> C137071; MOUSER (none) -> RC1210JR-07680RL
- TP1: value TestPoint_BMS -> TestPoint
- TP10, TP12, TP7: value TestPoint_SR_BMS -> TestPoint
- TP11: value TestPoint_IMD_Shutdown -> TestPoint
- TP2: value TestPoint_IMD -> TestPoint
- TP3: value TestPoint_BSPD -> TestPoint
- TP4: value TestPoint_BMS_Shutdown -> TestPoint
- TP6: value TestPoint_BSPD_Shutdown -> TestPoint
- U6: footprint (none) -> Package_DIP:DIP-14_W7.62mm
- renumbered U2 to U3
Connections:
- net +12V: now also PS1.22 (+VIN_1), PS1.23 (+VIN_2)
- net +5V: now also PS1.14 (+VOUT)
- net GND: now also PS1.16 (-VOUT)
- new net GNDPWR: PS1.2 (-VIN_1), PS1.3 (-VIN_2)
- no-connect marks 7 -> 9
